File: working/IBBC_0001/IBBC_0001.kicad_pcb (KiCad board)
At the start: 2 copper layers, 30 x 20 mm, 11 parts, among them J1 HEAD-I01-X-PI10-01 oom.lt/H10, J2 HEAD-I01-X-PI04-01 oom.lt/H4, J3 HEAD-JSTSH-X-PI04-RS oom.lt/H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, J4 HEAD-JSTSH-X-PI04-RS oom.lt/H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, U1 AP2112K-3.3, U2 ADXL343

Commit message: Workings.
Parts:
- removed H1, H2: MountingHole, MountingHole:MountingHole_3.2mm_M3
- removed J1: HEAD-I01-X-PI10-01 oom.lt/H10, Connector_PinHeader_2.54mm:PinHeader_1x10_P2.54mm_Vertical
- removed J2: HEAD-I01-X-PI04-01 oom.lt/H4, Connector_PinHeader_2.54mm:PinHeader_1x04_P2.54mm_Vertical
- removed J3, J4: HEAD-JSTSH-X-PI04-RS oom.lt/HSHR4, Connector_JST:JST_SH_SM04B-SRSS-TB_1x04-1MP_P1.00mm_Horizontal
- added U3: MODULE-CONN-BRBO-IBBC-SZ01, oomlout_OOMP_modules:MODULE-CONN-BRBO-IBBC-SZ01, F.Cu at (0.00, 0.00)
